File: KiCad/hot-air-reflow/hot-air-reflow.kicad_sch (KiCad schematic)
At the start: 27 parts, among them J1 Conn_01x04_Pin, P1 WJ127-5.0-2P, U1 STM32F103C8Tx, U2 TPS562201DDCR, Y1 8Mhz/12pF

Commit message: Record the current KiCad schematic and PCB so the board layout is in the repo.
Co-authored-by: Cursor <cursoragent@cursor.com>
Parts:
- added C10, C11, C12, C13, C14: 100nF/25V, Capacitor_SMD:C_0603_1608Metric, symbol Device:C
- added C15: 1uF/25V, Capacitor_SMD:C_0603_1608Metric, symbol Device:C
- C8, C9: value 15uF/50V -> 15pF/50V
- TP1, TP2, TP3: footprint (none) -> TestPoint:TestPoint_Pad_D1.5mm
Connections:
- net DBG_3.3V: now also C10.1, C11.1, C12.1, C13.1, C14.1, C15.1
- net ERROR_LED: now also U1.2 (PC13)
- net GND: now also P1.2, C10.2, C11.2, C12.2, C13.2, C14.2, C15.2; no longer P1.1
- net at C1.1, C2.1, C3.1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: now also P1.1; no longer P1.2
Other:
- moved on the sheet: C7, C8, C9, D1, D3, J1, R4, R6, TP1, U1, Y1
